Commit message: final uas

File: urdf/gazebo.xacro (robot description, xacro)
@@ -69,5 +69,5 @@
   <sensor type="ray" name="head_hokuyo_sensor">
     <pose>0 0 0 0 0 0</pose>
-    <visualize>false</visualize>
+    <visualize>true</visualize>
     <update_rate>20</update_rate>
     <ray>
@@ -97,5 +97,5 @@
   </sensor>
 </gazebo>
-<gazebo reference="camera">
+<!-- <gazebo reference="camera">
     <material>Gazebo/Green</material>
     <sensor type="camera" name="camera1">
@@ -128,4 +128,4 @@
       </plugin>
     </sensor>
-  </gazebo>
+  </gazebo> -->
 </robot>

File: urdf/m4wr.xacro (robot description, xacro)
@@ -15,5 +15,5 @@
     <collision name="collision_chassis">
       <geometry>
-        <box size="0.5 0.3 0.07"/>
+        <box size="0.5 0.3 0.1"/>
       </geometry>
     </collision>
@@ -21,5 +21,5 @@
       <origin rpy="0 0 0" xyz="0 0 0"/>
       <geometry>
-        <box size="0.5 0.3 0.07"/>
+        <box size="0.5 0.3 0.1"/>
       </geometry>
       <material name="blue"/>
@@ -28,15 +28,15 @@
   <!-- Create wheel right -->
   <xacro:link_steer_wheel name="front_link_right_wheel" />
-  <xacro:joint_steer_wheel name="front_joint_right_wheel"  child="front_link_right_wheel"  origin_xyz="0.15 0.15 0"  />
+  <xacro:joint_steer_wheel name="front_joint_right_wheel"  child="front_link_right_wheel"  origin_xyz="0.15 0.15 -0.1"  />
   <xacro:link_wheel name="back_link_right_wheel" />
-  <xacro:joint_wheel name="back_joint_right_wheel"  child="back_link_right_wheel"  origin_xyz="-0.15 0.15 0"  />
+  <xacro:joint_wheel name="back_joint_right_wheel"  child="back_link_right_wheel"  origin_xyz="-0.15 0.15 -0.1"  />
   <!-- Left Wheel link -->
   <xacro:link_steer_wheel name="front_link_left_wheel" />
-  <xacro:joint_steer_wheel name="front_joint_left_wheel"   child="front_link_left_wheel"   origin_xyz="0.15 -0.15 0"  />
+  <xacro:joint_steer_wheel name="front_joint_left_wheel"   child="front_link_left_wheel"   origin_xyz="0.15 -0.15 -0.1"  />
   <xacro:link_wheel name="back_link_left_wheel" />
-  <xacro:joint_wheel name="back_joint_left_wheel"   child="back_link_left_wheel"   origin_xyz="-0.15 -0.15 0"  />
-	 <xacro:property name="cameraSize" value="0.025"/>
-  <xacro:property name="cameraMass" value="0.1"/>
-  <link name="camera">
+  <xacro:joint_wheel name="back_joint_left_wheel"   child="back_link_left_wheel"   origin_xyz="-0.15 -0.15 -0.1"  />
+	<!-- <xacro:property name="cameraSize" value="0.025"/>
+  <xacro:property name="cameraMass" value="0.1"/> -->
+  <!-- <link name="camera">
     <collision>
       <origin xyz="0 0 0" rpy="0 0 0"/>
@@ -58,5 +58,5 @@
       <inertia ixx="1e-6" ixy="0" ixz="0" iyy="1e-6" iyz="0" izz="1e-6" />
     </inertial>
-  </link>
+  </link> -->
   <link name="sensor_laser">
     <inertial>
@@ -64,5 +64,5 @@
       <mass value="1" />
       <!-- < RANDOM INERTIA BELOW > -->
-      <inertia ixx="0.02" ixy="0" ixz="0" iyy="0.02" iyz="0" izz="0.02"/>
+      <xacro:cylinder_inertia mass="1" r="0.05" l="0.1" />
     </inertial>
     <visual>
@@ -74,5 +74,5 @@
     </visual>
     <collision>
-      <origin xyz="0 0 0" rpy="0 0 0"/>
+      <origin xyz="0.2 0 0.1" rpy="0 0 0"/>
       <geometry>
         <cylinder radius="0.05" length="0.1"/>
@@ -80,10 +80,10 @@
     </collision>
   </link>
-  <joint name="camera_joint" type="fixed">
+  <!-- <joint name="camera_joint" type="fixed">
     <axis xyz="0 1 0" />
     <origin xyz="0.265 0 0" rpy="0 0 0"/>
     <parent link="link_chassis"/>
     <child link="camera"/>
-  </joint>
+  </joint> -->
   <joint name="joint_sensor_laser" type="fixed">
     <origin xyz="0 0 0.085" rpy="0 0 0"/>

File: urdf/macro.xacro (robot description, xacro)
@@ -1,4 +1,4 @@
 <?xml version="1.0"?>
-<robot xmlns:xacro="http://www.ros.org/wiki/xacro">
+<robot xmlns:xacro="https://www.ros.org/wiki/xacro">
     <xacro:macro name="link_wheel" params="name">
       <link name="${name}">
@@ -63,9 +63,7 @@
       </joint>
     </xacro:macro>
-  <!--
 	<xacro:macro name="cylinder_inertia" params="mass r l">
     		<inertia ixx="${mass*(3*r*r+l*l)/12}" ixy = "0" ixz = "0"
                	 iyy="${mass*(3*r*r+l*l)/12}" iyz = "0" izz="${mass*(r*r)/2}" />
 	</xacro:macro>
-	<xacro:cylinder_inertia mass="1" r="0.05" l="0.1" />-->
 </robot>
